Commit message: Add stl file for backpack and ghostbuster ghost in urdf

File: urdf/backpack.urdf.xacro (robot description, xacro)
@@ -35,5 +35,40 @@
     <child link="lidar_link" />
   </joint>
-  <!-- Cameras -->
-  <!-- <xacro:include filename="$(find marmotte_description)/urdf/cameras.urdf.xacro"/> -->
+  <!-- Displaying CAD -->
+  <material name="grey">
+    <color rgba="${145/255} ${145/255} ${145/255} 1.0"/>
+  </material>
+  <material name="white">
+    <color rgba="${255/255} ${255/255} ${255/255} 1.0"/>
+  </material>
+  <xacro:property name="backpack_scale_CAD" value="0.001"/>
+  <xacro:property name="silouhette_scale_CAD" value="0.01"/>
+  <link name="backpack_CAD">
+    <visual>
+      <origin rpy="0 0 0" xyz="0 0 0"/>
+      <geometry>
+        <mesh filename="package://backpack_description/meshes/backpack.stl" scale="${backpack_scale_CAD} ${backpack_scale_CAD} ${backpack_scale_CAD}"/>
+      </geometry>
+      <material name="grey"/>
+    </visual>
+  </link>
+  <link name="silouhette_CAD">
+    <visual>
+      <origin rpy="0 0 0" xyz="0 0 0"/>
+      <geometry>
+        <mesh filename="package://backpack_description/meshes/StayPuftScan.stl" scale="${silouhette_scale_CAD} ${silouhette_scale_CAD} ${silouhette_scale_CAD}"/>
+      </geometry>
+      <material name="white"/>
+    </visual>
+  </link>
+  <joint name="backpack_CAD_base_joint" type="fixed">
+    <origin xyz="0 0 0" rpy="0 0 0" />
+    <parent link="base_link" />
+    <child link="backpack_CAD" />
+  </joint>
+  <joint name="silouhette_CAD_base_joint" type="fixed">
+    <origin xyz="0.7 0.95 -0.3" rpy="0 0 ${M_PI}" />
+    <parent link="base_link" />
+    <child link="silouhette_CAD" />
+  </joint>
 </robot>

Commit message: Format URDF, correct 'silhouette' and add footprint link

File: urdf/backpack.urdf.xacro (robot description, xacro)
@@ -1,12 +1,13 @@
 <?xml version="1.0"?>
 <robot name="backpack" xmlns:xacro="http://ros.org/wiki/xacro">
-  <xacro:property name="M_PI" value="3.14159"/>
+  <xacro:property name="M_PI" value="3.14159" />
   <!-- Links -->
-  <link name="base_link"/>
-  <link name="camera1_link"/>
-  <link name="camera2_link"/>
-  <link name="gps_link"/>
-  <link name="imu_link"/>
-  <link name="lidar_link"/>
+  <link name="base_link" />
+  <link name="camera1_link" />
+  <link name="camera2_link" />
+  <link name="gps_link" />
+  <link name="imu_link" />
+  <link name="lidar_link" />
+  <link name="base_footprint" />
   <!-- Joints -->
   <joint name="camera1_base_joint" type="fixed">
@@ -37,27 +38,29 @@
   <!-- Displaying CAD -->
   <material name="grey">
-    <color rgba="${145/255} ${145/255} ${145/255} 1.0"/>
+    <color rgba="${145/255} ${145/255} ${145/255} 1.0" />
   </material>
   <material name="white">
-    <color rgba="${255/255} ${255/255} ${255/255} 1.0"/>
+    <color rgba="${255/255} ${255/255} ${255/255} 1.0" />
   </material>
-  <xacro:property name="backpack_scale_CAD" value="0.001"/>
-  <xacro:property name="silouhette_scale_CAD" value="0.01"/>
+  <xacro:property name="backpack_scale_CAD" value="0.001" />
+  <xacro:property name="silhouette_scale_CAD" value="0.01" />
   <link name="backpack_CAD">
     <visual>
-      <origin rpy="0 0 0" xyz="0 0 0"/>
+      <origin rpy="0 0 0" xyz="0 0 0" />
       <geometry>
-        <mesh filename="package://backpack_description/meshes/backpack.stl" scale="${backpack_scale_CAD} ${backpack_scale_CAD} ${backpack_scale_CAD}"/>
+        <mesh filename="package://backpack_description/meshes/backpack.stl"
+          scale="${backpack_scale_CAD} ${backpack_scale_CAD} ${backpack_scale_CAD}" />
       </geometry>
-      <material name="grey"/>
+      <material name="grey" />
     </visual>
   </link>
-  <link name="silouhette_CAD">
+  <link name="silhouette_CAD">
     <visual>
-      <origin rpy="0 0 0" xyz="0 0 0"/>
+      <origin rpy="0 0 0" xyz="0 0 0" />
       <geometry>
-        <mesh filename="package://backpack_description/meshes/StayPuftScan.stl" scale="${silouhette_scale_CAD} ${silouhette_scale_CAD} ${silouhette_scale_CAD}"/>
+        <mesh filename="package://backpack_description/meshes/StayPuftScan.stl"
+          scale="${silhouette_scale_CAD} ${silhouette_scale_CAD} ${silhouette_scale_CAD}" />
       </geometry>
-      <material name="white"/>
+      <material name="white" />
     </visual>
   </link>
@@ -67,8 +70,13 @@
     <child link="backpack_CAD" />
   </joint>
-  <joint name="silouhette_CAD_base_joint" type="fixed">
+  <joint name="silhouette_CAD_base_joint" type="fixed">
     <origin xyz="0.7 0.95 -0.3" rpy="0 0 ${M_PI}" />
     <parent link="base_link" />
-    <child link="silouhette_CAD" />
+    <child link="silhouette_CAD" />
+  </joint>
+  <joint name="footprint_joint" type="fixed">
+    <origin xyz="-0.298971 0 -0.3" rpy="0 0 0" />
+    <parent link="base_link" />
+    <child link="base_footprint" />
   </joint>
 </robot>

Commit message: Add base_footprint ros1

File: urdf/backpack.urdf.xacro (robot description, xacro)
@@ -4,9 +4,10 @@
   <!-- Links -->
   <link name="base_link"/>
+  <link name="base_footprint" />
   <link name="camera1_link"/>
   <link name="camera2_link"/>
+  <link name="lidar_link"/>
+  <link name="imu_link"/>
   <link name="gps_link"/>
-  <link name="imu_link"/>
-  <link name="lidar_link"/>
   <!-- Joints -->
   <joint name="camera1_base_joint" type="fixed">
@@ -43,5 +44,5 @@
   </material>
   <xacro:property name="backpack_scale_CAD" value="0.001"/>
-  <xacro:property name="silouhette_scale_CAD" value="0.01"/>
+  <xacro:property name="silhouette_scale_CAD" value="0.01"/>
   <link name="backpack_CAD">
     <visual>
@@ -53,9 +54,9 @@
     </visual>
   </link>
-  <link name="silouhette_CAD">
+  <link name="silhouette_CAD">
     <visual>
       <origin rpy="0 0 0" xyz="0 0 0"/>
       <geometry>
-        <mesh filename="package://backpack_description/meshes/StayPuftScan.stl" scale="${silouhette_scale_CAD} ${silouhette_scale_CAD} ${silouhette_scale_CAD}"/>
+        <mesh filename="package://backpack_description/meshes/StayPuftScan.stl" scale="${silhouette_scale_CAD} ${silhouette_scale_CAD} ${silhouette_scale_CAD}"/>
       </geometry>
       <material name="white"/>
@@ -67,8 +68,13 @@
     <child link="backpack_CAD" />
   </joint>
-  <joint name="silouhette_CAD_base_joint" type="fixed">
+  <joint name="silhouette_CAD_base_joint" type="fixed">
     <origin xyz="0.7 0.95 -0.3" rpy="0 0 ${M_PI}" />
     <parent link="base_link" />
-    <child link="silouhette_CAD" />
+    <child link="silhouette_CAD" />
+  </joint>
+  <joint name="footprint__base_joint" type="fixed">
+    <origin xyz="-0.298971 0 -0.3" rpy="0 0 0" />
+    <parent link="base_link" />
+    <child link="base_footprint" />
   </joint>
 </robot>

Commit message: Change position of base_link to have it in the center of the body

File: urdf/backpack.urdf.xacro (robot description, xacro)
@@ -4,4 +4,5 @@
   <!-- Links -->
   <link name="base_link"/>
+  <link name="sensor_rack"/>
   <link name="base_footprint" />
   <link name="camera1_link"/>
@@ -11,27 +12,32 @@
   <link name="gps_link"/>
   <!-- Joints -->
+  <joint name="sensor_rack_base_joint" type="fixed">
+    <origin xyz="0.33 0 0" rpy="0 0 0" />
+    <parent link="base_link" />
+    <child link="sensor_rack" />
+  </joint>
   <joint name="camera1_base_joint" type="fixed">
     <origin xyz="-0.030688 0.090001 0.056917" rpy="-1.74533 0 -${M_PI/2}" />
-    <parent link="base_link" />
+    <parent link="sensor_rack" />
     <child link="camera1_link" />
   </joint>
   <joint name="camera2_base_joint" type="fixed">
     <origin xyz="-0.030688 -0.090001 0.056917" rpy="-1.74533 0 -${M_PI/2}" />
-    <parent link="base_link" />
+    <parent link="sensor_rack" />
     <child link="camera2_link" />
   </joint>
   <joint name="gps_base_joint" type="fixed">
     <origin xyz="-0.597942 0.004732 0.719853" rpy="0 0.0349066 0" />
-    <parent link="base_link" />
+    <parent link="sensor_rack" />
     <child link="gps_link" />
   </joint>
   <joint name="imu_base_joint" type="fixed">
     <origin xyz="0.012516 0.00245 0.032" rpy="0 0 0" />
-    <parent link="base_link" />
+    <parent link="sensor_rack" />
     <child link="imu_link" />
   </joint>
   <joint name="lidar_base_joint" type="fixed">
     <origin xyz="0 0 0.145700" rpy="0 0 0" />
-    <parent link="base_link" />
+    <parent link="sensor_rack" />
     <child link="lidar_link" />
   </joint>
@@ -65,15 +71,15 @@
   <joint name="backpack_CAD_base_joint" type="fixed">
     <origin xyz="0 0 0" rpy="0 0 0" />
-    <parent link="base_link" />
+    <parent link="sensor_rack" />
     <child link="backpack_CAD" />
   </joint>
   <joint name="silhouette_CAD_base_joint" type="fixed">
     <origin xyz="0.7 0.95 -0.3" rpy="0 0 ${M_PI}" />
-    <parent link="base_link" />
+    <parent link="sensor_rack" />
     <child link="silhouette_CAD" />
   </joint>
-  <joint name="footprint__base_joint" type="fixed">
+  <joint name="footprint_base_joint" type="fixed">
     <origin xyz="-0.298971 0 -0.3" rpy="0 0 0" />
-    <parent link="base_link" />
+    <parent link="sensor_rack" />
     <child link="base_footprint" />
   </joint>

Commit message: Update backpack.urdf.xacro
Lidar-IMU calibrated value

File: urdf/backpack.urdf.xacro (robot description, xacro)
@@ -32,5 +32,5 @@
   </joint>
   <joint name="lidar_base_joint" type="fixed">
-    <origin xyz="0 0 0.145700" rpy="0 0 0" />
+    <origin xyz="0 0 0.145700" rpy="0 -0.015 0" />
     <parent link="base_link" />
     <child link="lidar_link" />

Commit message: Update backpack.urdf.xacro
Update calibrated lidar pitch value

File: urdf/backpack.urdf.xacro (robot description, xacro)
@@ -32,5 +32,5 @@
   </joint>
   <joint name="lidar_base_joint" type="fixed">
-    <origin xyz="0 0 0.145700" rpy="0 -0.015 0" />
+    <origin xyz="0 0 0.145700" rpy="0 -0.018 0" />
     <parent link="base_link" />
     <child link="lidar_link" />

Commit message: Backpack description for Congress mapping for an Ulaval event

File: urdf/backpack.urdf.xacro (robot description, xacro)
@@ -32,5 +32,9 @@
   </joint>
   <joint name="lidar_base_joint" type="fixed">
-    <origin xyz="0 0 0.145700" rpy="0 -0.018 0" />
+  <!-- There seem to be two configurations of pitch angles that work for most rosbags:
+        -0.011 and
+        -0.018.
+        0.00183159 for Journal paper 7am backpack rosbag -->
+    <origin xyz="0 0 0.145700" rpy="0 -0.003 0" />
     <parent link="base_link" />
     <child link="lidar_link" />
